Commit message: updates

File: obstacle2/urdf/obstacle2.urdf (robot description, URDF)
Before this commit: robot track2, 1 links, 0 joints
Links:
- removed link base_link
- added link cube, mass 1000; collision mesh filename=package://obstacle2/meshes/cube.STL; visual mesh filename=package://obstacle2/meshes/cube.STL
