Commit message: updates

File: track2/urdf/track2.urdf (robot description, URDF)
Before this commit: robot track, 1 links, 0 joints
Links:
- link base_link: mass 0.00606225780461374 -> 122116.506904259; geometry collision mesh filename=package://track2/meshes/base_link.STL; visual mesh filename=package://track2/meshes/base_link.STL

Commit message: updates

File: track2/urdf/track2.urdf (robot description, URDF)
Before this commit: robot track3, 1 links, 0 joints
Links:
- link base_link: mass 155904.571726482 -> 147534.352794364; geometry collision mesh filename=package://track2/meshes/base_link.STL; visual mesh filename=package://track2/meshes/base_link.STL
